File: projects/nrfl15_usb_dongle/nrfl15_usb_dongle.kicad_sch (KiCad schematic)
At the start: 0 parts

Commit message: Add nrfl15 usb dongle project
Parts:
- added C1: 10n, Capacitor_SMD:C_0402_1005Metric, symbol Device:C_Small
- added C2, C3: 4.7u, Capacitor_SMD:C_0603_1608Metric, symbol Device:C_Small
- added C4, C5: 100n, Capacitor_SMD:C_0402_1005Metric, symbol Device:C_Small
- added FB1: MI0805K601R-10, Inductor_SMD:L_0805_2012Metric, symbol Device:FerriteBead_Small
- added J1: USB_A, Connector_USB:USB_A_Molex_48037-2200_Horizontal, symbol Connector:USB_A
- added J2: Conn_ARM_JTAG_SWD_10, Connector_PinHeader_1.27mm:PinHeader_2x05_P1.27mm_Vertical_SMD, symbol Connector:Conn_ARM_JTAG_SWD_10
- added R1, R2: 27, Resistor_SMD:R_0402_1005Metric, symbol Device:R_Small_US
- added R3: 1k, Resistor_SMD:R_0402_1005Metric, symbol Device:R_Small_US
- added U1: BM15M, bobby:BM15M, symbol bobby:BM15M
- added U2: FT234XD, Package_DFN_QFN:WDFN-12-1EP_3x3mm_P0.45mm_EP1.7x2.5mm, symbol Interface_USB:FT234XD
Connections:
- new net: R1.2, U2.12 (USBDP)
- new net: R2.1, U2.1 (USBDM)
- new net +3.3V: C3.1, C5.1, J2.1 (VTref), R3.1, U1.B8 (VDD), U1.C8 (VDD), U2.3 (3V3OUT), U2.9 (VCCIO)
- new net +5V: C2.1, FB1.2, U2.4 (VCC)
- new net D+: J1.3 (D+), R1.1
- new net D-: J1.2 (D-), R2.2
- new net GND: C1.2, C2.2, C3.2, C4.2, C5.2, J1.4 (GND), J1.5 (Shield), J2.3 (GND), J2.5 (GND), J2.9 (GNDDetect), U1.A1 (GND), U1.A9 (GND), U1.B1 (GND), U1.B7 (GND), U1.B9 (GND), U1.D1 (GND), U1.E1 (GND), U1.F1 (GND), U1.H8 (GND), U2.13 (GND), U2.5 (GND)
- new net NRF_RX: U1.H9 (P2.00), U2.7 (TXD/D0)
- new net NRF_TX: U1.J8 (P2.02), U2.10 (RXD/D1)
- new net SWDCLK: J2.4 (SWCLK/TCK), U1.K3 (SWDCLK)
- new net SWDIO: J2.2 (SWDIO/TMS), U1.J3 (SWDIO)
- new net VBUS: C1.1, FB1.1, J1.1 (VBUS)
- new net ~{RESET}: C4.1, J2.10 (~{RESET}), R3.2, U1.G2 (~{Reset})
- no-connect marks 0 -> 35
Other:
- note added: "BLE Module"
- note added: "Close to 3V3OUT"
- note added: "Close to VCC"
- note added: "Module Decoupling"
- note added: "Place as close to USB connector as possible"
- note added: "Power Sources"
- note added: "Reset Circuit"
- note added: "SWD Connector"
- note added: "UART to USB"
- note added: "UART to USB Decoupling"
- note added: "USB Connector"
